File: Power_rails.kicad_sch (KiCad schematic)
At the start: 75 parts

Commit message: first iteration of sdram
Fanout completed, started tracing towards the chip
Parts:
- removed R27: 0 Ohm, symbol Device:R_Small
- C21, C22, C23, C24, C25, C26, C27, C28, C29, C30, C31, C32, C33, C34, C35, C36, C37, C38, C39, C40, C41, C42, C43, C44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: footprint Capacitor_SMD:C_0603_1608Metric_Pad1.08x0.95mm_HandSolder -> Capacitor_SMD:C_0402_1005Metric_Pad0.74x0.62mm_HandSolder
