File: config_reset.kicad_sch (KiCad schematic)
At the start: 20 parts, among them U1 NX1H35 PBGA625, U6 M95P32-IXMNT/E, Y2 LFSPXO025225_25MHz

Commit message: first iteration of sdram
Fanout completed, started tracing towards the chip
Parts:
- C14: footprint Capacitor_SMD:C_0603_1608Metric_Pad1.08x0.95mm_HandSolder -> Capacitor_SMD:C_0402_1005Metric_Pad0.74x0.62mm_HandSolder
Changed lines of the file:
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@@
 			)
 		)
-		(property "Footprint" "Capacitor_SMD:C_0603_1608Metric_Pad1.08x0.95mm_HandSolder"
+		(property "Footprint" "Capacitor_SMD:C_0402_1005Metric_Pad0.74x0.62mm_HandSolder"
 			(at 142.24 166.37 0)
 			(effects
