File: PCB_Project.kicad_pcb (KiCad board)
At the start: 8 copper layers, 152.4 x 101.6 mm, 133 parts, among them J2 DF9-41P-1V32, J3 DF9-CFG-SPW1, J5 DF9-41P-1V32, J6 DF9-41P-1V32, U1 NX1H35 PBGA625, U2 CY15B108QN-40SXI, U3 M95P32-IXMNT/E, U4 CY15B108QN-40SXI, U5 AS4C8M32S-6TIN, U6 M95P32-IXMNT/E, U7 TPS3828-33DBVR, Y2 LFSPXO025225_25MHz

Commit message: SDRAM, bank5
last iteration of sdram. max optimization routing and space wise. Traced 2 frams to Bank 5. Fanout of bank 5 for DF9
Parts:
- removed J5, J6: DF9-41P-1V32, DataHub_Footprints:DF941P1V32
- added R21: 0 Ohm, Resistor_SMD:R_0402_1005Metric_Pad0.72x0.64mm_HandSolder, F.Cu at (118.6, 36.3)
- added R22: 0 Ohm, Resistor_SMD:R_0402_1005Metric_Pad0.72x0.64mm_HandSolder, F.Cu at (118.6, 38.3)
- added R23: 0 Ohm, Resistor_SMD:R_0402_1005Metric_Pad0.72x0.64mm_HandSolder, F.Cu at (118.6, 40.3)
- added R24: 0 Ohm, Resistor_SMD:R_0402_1005Metric_Pad0.72x0.64mm_HandSolder, F.Cu at (118.6, 42.3)
- added R25: 0 Ohm, Resistor_SMD:R_0402_1005Metric_Pad0.72x0.64mm_HandSolder, F.Cu at (118.6, 44.3)
- added R26: 0 Ohm, Resistor_SMD:R_0402_1005Metric_Pad0.72x0.64mm_HandSolder, F.Cu at (118.6, 46.3)
- added R28: 0 Ohm, Resistor_SMD:R_0402_1005Metric_Pad0.72x0.64mm_HandSolder, F.Cu at (118.6, 48.3)
- added R29: 0 Ohm, Resistor_SMD:R_0402_1005Metric_Pad0.72x0.64mm_HandSolder, F.Cu at (118.6, 50.3)
- added R30: 0 Ohm, Resistor_SMD:R_0402_1005Metric_Pad0.72x0.64mm_HandSolder, F.Cu at (118.6, 52.3)
- added REF**: 21-0140L_T1655-3_MXM, DataHub_Footprints:MAX8556, F.Cu at (163.9, 78.7)
- added REF**: Edge&Holes_DH+, DataHub_Footprints:Edge&Holes_DH+, F.Cu at (158.3, 102.1)
- C15, C16, C17, C18, C19, C20, C22, C23, C24, C80, C84, C85, C86, C88, C89, C90, J2, J3, U4: moved to B.Cu
- L1, L2, L3, L4, L5: footprint Inductor_SMD:L_0805_2012Metric_Pad1.05x1.20mm_HandSolder -> Inductor_SMD:L_0402_1005Metric_Pad0.77x0.64mm_HandSolder
- R1, R10, R11, R12, R13, R14, R15, R16, R17, R18, R19, R2, R3, R31, R32, R4, R6, R7, R8, R9: footprint Resistor_SMD:R_0603_1608Metric_Pad0.98x0.95mm_HandSolder -> Resistor_SMD:R_0402_1005Metric_Pad0.72x0.64mm_HandSolder
- R5: footprint Resistor_SMD:R_0603_1608Metric_Pad0.98x0.95mm_HandSolder -> Resistor_SMD:R_0402_1005Metric_Pad0.72x0.64mm_HandSolder; moved to B.Cu
- moved REF** 127.0 mm to (-111.1, 113.8)
- moved C13 100.8 mm to (183.1, 135.5)
- moved R2 97.4 mm to (183.1, 138.5)
- moved J2 95.4 mm to (181.2, 97.6), turned to -90 degrees
- moved C17 80.9 mm to (171.4, 124.4), turned to 90 degrees
- moved R5 77.9 mm to (170.7, 128.5), turned to -90 degrees
- moved C15 76.4 mm to (170.2, 116.9), turned to 90 degrees
- moved R4 68.2 mm to (169.3, 113.7), turned to 180 degrees
- moved C9 68.2 mm to (139.4, 103.0), turned to 180 degrees
- moved C89 65.4 mm to (161.8, 112.8), turned to -90 degrees
- moved C7 63.4 mm to (139.4, 106.0), turned to 180 degrees
- moved C90 61.5 mm to (164.9, 112.8), turned to -90 degrees
- moved C8 61.2 mm to (139.4, 104.5), turned to 180 degrees
- moved C88 58.5 mm to (156.8, 102.6), turned to 180 degrees
- moved L3 57.0 mm to (139.4, 107.5)
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Connections:
- C76 pad 1: VDDIO_0 -> VDDIO_8
- C77 pad 1: VDDIO_0 -> VDDIO_8
- C78 pad 1: VDDIO_0 -> VDDIO_8
- D2 pad 2: /DF9_CFG-SPW/RST_N -> RST_N
- J3 pad 5: /DF9_CFG-SPW/RST_N -> RST_N
- R15 pad 2: /DF9_CFG-SPW/RST_N -> RST_N
- U1 pad AA10: unconnected-(U1C-IO_B3D10P-PadAA10) -> /04_FPGA_Banks2_3_SDRAM/SDRAM_DQ17
- U1 pad AA11: /04_FPGA_Banks2_3_SDRAM/SDRAM_DQ22 -> /04_FPGA_Banks2_3_SDRAM/SDRAM_DQ20
- U1 pad AA12: /04_FPGA_Banks2_3_SDRAM/SDRAM_A8 -> /04_FPGA_Banks2_3_SDRAM/SDRAM_DQ26
- U1 pad AA18: /05_FPGA_Bank5_SPI/EEPROM_MOSI -> unconnected-(U1D-IO_B5D13P_DQS_SWSO-PadAA18)
- U1 pad AA19: /05_FPGA_Bank5_SPI/FRAM1_MOSI -> unconnected-(U1D-IO_B5D10N_DQ-PadAA19)
- U1 pad AA20: /05_FPGA_Bank5_SPI/FRAM2_MOSI -> unconnected-(U1D-IO_B5D10P-PadAA20)
- U1 pad AA22: /05_FPGA_Bank5_SPI/EEPROM_WP_N -> unconnected-(U1D-IO_B5D04N_DQ_SWSI-PadAA22)
- U1 pad AA3: /04_FPGA_Banks2_3_SDRAM/SDRAM_DQ0 -> /04_FPGA_Banks2_3_SDRAM/SDRAM_DQ15
- U1 pad AA5: /04_FPGA_Banks2_3_SDRAM/SDRAM_A2 -> /04_FPGA_Banks2_3_SDRAM/SDRAM_DQ5
- U1 pad AA6: /04_FPGA_Banks2_3_SDRAM/SDRAM_DQ9 -> /04_FPGA_Banks2_3_SDRAM/SDRAM_WE_N
- U1 pad AA7: /04_FPGA_Banks2_3_SDRAM/SDRAM_DQ31 -> /04_FPGA_Banks2_3_SDRAM/SDRAM_CKE
- U1 pad AA8: /04_FPGA_Banks2_3_SDRAM/SDRAM_DQ17 -> /04_FPGA_Banks2_3_SDRAM/SDRAM_A0
- U1 pad AA9: /04_FPGA_Banks2_3_SDRAM/SDRAM_CLK -> /04_FPGA_Banks2_3_SDRAM/SDRAM_A5
- U1 pad AB10: /04_FPGA_Banks2_3_SDRAM/SDRAM_DQ20 -> /04_FPGA_Banks2_3_SDRAM/SDRAM_A1
- U1 pad AB11: unconnected-(U1C-IO_B3D06N_CAL-PadAB11) -> /04_FPGA_Banks2_3_SDRAM/SDRAM_A2
- U1 pad AB12: /04_FPGA_Banks2_3_SDRAM/SDRAM_DQ23 -> /04_FPGA_Banks2_3_SDRAM/SDRAM_DQ27
- U1 pad AB19: /05_FPGA_Bank5_SPI/EEPROM_CLK -> unconnected-(U1D-IO_B5D15N_DQ_SWSI-PadAB19)
- U1 pad AB20: /05_FPGA_Bank5_SPI/FRAM1_CLK -> unconnected-(U1D-IO_B5D09N-PadAB20)
- U1 pad AB22: /05_FPGA_Bank5_SPI/EEPROM_MISO -> unconnected-(U1D-IO_B5D04P_DQ_SWSI-PadAB22)
- U1 pad AB3: /04_FPGA_Banks2_3_SDRAM/SDRAM_DQ1 -> /04_FPGA_Banks2_3_SDRAM/SDRAM_DQ4
- U1 pad AB4: /04_FPGA_Banks2_3_SDRAM/SDRAM_DQ11 -> /04_FPGA_Banks2_3_SDRAM/SDRAM_DQ6
- U1 pad AB5: /04_FPGA_Banks2_3_SDRAM/SDRAM_DQM2 -> /04_FPGA_Banks2_3_SDRAM/SDRAM_DQ10
- U1 pad AB6: /04_FPGA_Banks2_3_SDRAM/SDRAM_DQ8 -> /04_FPGA_Banks2_3_SDRAM/SDRAM_CAS_N
- U1 pad AB7: /04_FPGA_Banks2_3_SDRAM/SDRAM_DQ30 -> /04_FPGA_Banks2_3_SDRAM/SDRAM_BA0
- U1 pad AB8: /04_FPGA_Banks2_3_SDRAM/SDRAM_DQ18 -> /04_FPGA_Banks2_3_SDRAM/SDRAM_A10
- U1 pad AB9: /04_FPGA_Banks2_3_SDRAM/SDRAM_DQ6 -> /04_FPGA_Banks2_3_SDRAM/SDRAM_A7
- U1 pad AC10: unconnected-(U1C-IO_B3D06P_DQ-PadAC10) -> /04_FPGA_Banks2_3_SDRAM/SDRAM_DQ16
- U1 pad AC11: /04_FPGA_Banks2_3_SDRAM/SDRAM_DQ25 -> /04_FPGA_Banks2_3_SDRAM/SDRAM_DQ30
- U1 pad AC12: /04_FPGA_Banks2_3_SDRAM/SDRAM_DQ24 -> /04_FPGA_Banks2_3_SDRAM/SDRAM_DQ29
- U1 pad AC19: /05_FPGA_Bank5_SPI/FRAM2_CLK -> unconnected-(U1D-IO_B5D15P_DQ_SWSI-PadAC19)
- U1 pad AC2: /04_FPGA_Banks2_3_SDRAM/SDRAM_DQ15 -> /04_FPGA_Banks2_3_SDRAM/SDRAM_DQ11
- U1 pad AC20: /05_FPGA_Bank5_SPI/FRAM1_MISO -> /05_FPGA_Bank5_SPI/FRAM2_MISO
- U1 pad AC21: /05_FPGA_Bank5_SPI/FRAM1_CS_N -> /05_FPGA_Bank5_SPI/FRAM1_CLK
- U1 pad AC22: /05_FPGA_Bank5_SPI/FRAM2_MISO -> unconnected-(U1D-IO_B5D06P_DQ-PadAC22)
- U1 pad AC23: /05_FPGA_Bank5_SPI/FRAM2_CS_N -> /05_FPGA_Bank5_SPI/FRAM2_CLK
- U1 pad AC24: /05_FPGA_Bank5_SPI/EEPROM_CS_N -> /05_FPGA_Bank5_SPI/FRAM1_MISO
- U1 pad AC3: /04_FPGA_Banks2_3_SDRAM/SDRAM_DQ14 -> /04_FPGA_Banks2_3_SDRAM/SDRAM_DQ9
- U1 pad AC4: /04_FPGA_Banks2_3_SDRAM/SDRAM_DQ10 -> /04_FPGA_Banks2_3_SDRAM/SDRAM_DQ7
- U1 pad AC5: /04_FPGA_Banks2_3_SDRAM/SDRAM_A11 -> /04_FPGA_Banks2_3_SDRAM/SDRAM_DQM0
- U1 pad AC6: /04_FPGA_Banks2_3_SDRAM/SDRAM_BA0 -> /04_FPGA_Banks2_3_SDRAM/SDRAM_RAS_N
- U1 pad AC7: /04_FPGA_Banks2_3_SDRAM/SDRAM_DQ19 -> /04_FPGA_Banks2_3_SDRAM/SDRAM_CS_N
- U1 pad AC8: /04_FPGA_Banks2_3_SDRAM/SDRAM_DQ7 -> /04_FPGA_Banks2_3_SDRAM/SDRAM_A9
- U1 pad AC9: /04_FPGA_Banks2_3_SDRAM/SDRAM_DQ21 -> /04_FPGA_Banks2_3_SDRAM/SDRAM_A4
- U1 pad AD1: /04_FPGA_Banks2_3_SDRAM/SDRAM_BA1 -> /04_FPGA_Banks2_3_SDRAM/SDRAM_DQ14
- U1 pad AD11: /04_FPGA_Banks2_3_SDRAM/SDRAM_DQ27 -> /04_FPGA_Banks2_3_SDRAM/SDRAM_A3
- U1 pad AD22: unconnected-(U1D-IO_B5D05N_DQ-PadAD22) -> /05_FPGA_Bank5_SPI/FRAM2_MOSI
- U1 pad AD25: unconnected-(U1D-IO_B5D01N_DQ_SWDO-PadAD25) -> /05_FPGA_Bank5_SPI/FRAM2_CS_N
- U1 pad AD4: /04_FPGA_Banks2_3_SDRAM/SDRAM_DQ13 -> /04_FPGA_Banks2_3_SDRAM/SDRAM_DQ8
- U1 pad AD9: /04_FPGA_Banks2_3_SDRAM/SDRAM_DQM0 -> /04_FPGA_Banks2_3_SDRAM/SDRAM_A6
- U1 pad AE1: /04_FPGA_Banks2_3_SDRAM/SDRAM_A10 -> /04_FPGA_Banks2_3_SDRAM/SDRAM_DQ12
- U1 pad AE11: /04_FPGA_Banks2_3_SDRAM/SDRAM_DQ26 -> /04_FPGA_Banks2_3_SDRAM/SDRAM_DQ31
- U1 pad AE22: unconnected-(U1D-IO_B5D05P_DQ-PadAE22) -> /05_FPGA_Bank5_SPI/FRAM1_MOSI
- U1 pad AE25: unconnected-(U1D-IO_B5D01P_DQ_SWDO-PadAE25) -> /05_FPGA_Bank5_SPI/FRAM1_CS_N
- U1 pad AE4: /04_FPGA_Banks2_3_SDRAM/SDRAM_DQ12 -> /04_FPGA_Banks2_3_SDRAM/SDRAM_DQM1
- U1 pad AE8: /04_FPGA_Banks2_3_SDRAM/SDRAM_WE_N -> /04_FPGA_Banks2_3_SDRAM/SDRAM_A8
- U1 pad F1: VDDIO_0 -> GND
- U1 pad F25: GND -> VDDIO_8
- U1 pad G21: unconnected-(U1E-IO_B8D02N-PadG21) -> /03_FPGA_Bank0_Dsu_UART/DSU_TX
- U1 pad G22: unconnected-(U1E-IO_B8D02P_CLK1-PadG22) -> /03_FPGA_Bank0_Dsu_UART/LD_USER1
- U1 pad G24: unconnected-(U1E-IO_B8D03N-PadG24) -> /03_FPGA_Bank0_Dsu_UART/JULIET_TX
- U1 pad H1: /03_FPGA_Bank0_Dsu_UART/LD_USER1 -> unconnected-(U1A-IO_B0D01P-PadH1)
- U1 pad H19: unconnected-(U1E-IO_B8D04N-PadH19) -> /03_FPGA_Bank0_Dsu_UART/LD_USER2
- U1 pad H2: /03_FPGA_Bank0_Dsu_UART/DSU_TX -> unconnected-(U1A-IO_B0D01N-PadH2)
- U1 pad H20: unconnected-(U1E-IO_B8D04P-PadH20) -> /03_FPGA_Bank0_Dsu_UART/LD_USER3
- U1 pad H25: unconnected-(U1E-IO_B8D11N-PadH25) -> /03_FPGA_Bank0_Dsu_UART/JULIET_RX
- U1 pad H7: /03_FPGA_Bank0_Dsu_UART/DSU_RX -> unconnected-(U1A-IO_B0D11N-PadH7)
- U1 pad J1: VDDIO_0 -> GND
- U1 pad J25: GND -> VDDIO_8
- U1 pad J4: /03_FPGA_Bank0_Dsu_UART/JULIET_TX -> unconnected-(U1A-IO_B0D02N-PadJ4)
- U1 pad J5: /03_FPGA_Bank0_Dsu_UART/LD_USER3 -> unconnected-(U1A-IO_B0D03P-PadJ5)
- U1 pad J6: /03_FPGA_Bank0_Dsu_UART/LD_USER2 -> unconnected-(U1A-IO_B0D03N-PadJ6)
- U1 pad J8: /03_FPGA_Bank0_Dsu_UART/JULIET_RX -> unconnected-(U1A-IO_B0D10N-PadJ8)
- U1 pad K18: GND -> VDDIO_8
- U1 pad K22: unconnected-(U1E-IO_B8D12N-PadK22) -> /03_FPGA_Bank0_Dsu_UART/DSU_RX
- U1 pad L6: /02_FPGA_Config_JTAG_Bitstream_Reset/RST_N -> RST_N
- U1 pad L9: VDDIO_0 -> GND
- U1 pad U10: /04_FPGA_Banks2_3_SDRAM/SDRAM_A3 -> unconnected-(U1C-IO_B2D08P_CLK0-PadU10)
- U1 pad U11: /04_FPGA_Banks2_3_SDRAM/SDRAM_CKE -> unconnected-(U1C-IO_B3D08N-PadU11)
- U1 pad U9: /04_FPGA_Banks2_3_SDRAM/SDRAM_A4 -> unconnected-(U1C-IO_B2D08N-PadU9)
- U1 pad V10: /04_FPGA_Banks2_3_SDRAM/SDRAM_DQ29 -> /04_FPGA_Banks2_3_SDRAM/SDRAM_DQ25
- U1 pad V11: /04_FPGA_Banks2_3_SDRAM/SDRAM_A9 -> /04_FPGA_Banks2_3_SDRAM/SDRAM_DQ24
- U1 pad V12: /04_FPGA_Banks2_3_SDRAM/SDRAM_A5 -> /04_FPGA_Banks2_3_SDRAM/SDRAM_DQ23
- U1 pad V8: /04_FPGA_Banks2_3_SDRAM/SDRAM_DQM3 -> unconnected-(U1C-IO_B2D09N-PadV8)
- U1 pad W11: /04_FPGA_Banks2_3_SDRAM/SDRAM_CAS_N -> /04_FPGA_Banks2_3_SDRAM/SDRAM_DQM2
- U1 pad W12: /04_FPGA_Banks2_3_SDRAM/SDRAM_A6 -> /04_FPGA_Banks2_3_SDRAM/SDRAM_DQ22
- U1 pad W6: /04_FPGA_Banks2_3_SDRAM/SDRAM_DQ4 -> /04_FPGA_Banks2_3_SDRAM/SDRAM_DQ0
- U1 pad W7: /04_FPGA_Banks2_3_SDRAM/SDRAM_A0 -> /04_FPGA_Banks2_3_SDRAM/SDRAM_DQ1
- U1 pad W8: /04_FPGA_Banks2_3_SDRAM/SDRAM_CS_N -> /04_FPGA_Banks2_3_SDRAM/SDRAM_A11
- U1 pad Y10: unconnected-(U1C-IO_B3D10N_DQ-PadY10) -> /04_FPGA_Banks2_3_SDRAM/SDRAM_DQ19
- U1 pad Y11: /04_FPGA_Banks2_3_SDRAM/SDRAM_RAS_N -> /04_FPGA_Banks2_3_SDRAM/SDRAM_DQ18
- U1 pad Y12: /04_FPGA_Banks2_3_SDRAM/SDRAM_A7 -> /04_FPGA_Banks2_3_SDRAM/SDRAM_DQ21
- U1 pad Y18: /05_FPGA_Bank5_SPI/EEPROM_HOLD_N -> unconnected-(U1D-IO_B5D13N_DQS_SWSO-PadY18)
- U1 pad Y5: /04_FPGA_Banks2_3_SDRAM/SDRAM_DQ3 -> /04_FPGA_Banks2_3_SDRAM/SDRAM_DQ13
- U1 pad Y6: /04_FPGA_Banks2_3_SDRAM/SDRAM_DQ5 -> /04_FPGA_Banks2_3_SDRAM/SDRAM_DQ3
- U1 pad Y7: /04_FPGA_Banks2_3_SDRAM/SDRAM_A1 -> /04_FPGA_Banks2_3_SDRAM/SDRAM_CLK
- U1 pad Y8: /04_FPGA_Banks2_3_SDRAM/SDRAM_DQ16 -> /04_FPGA_Banks2_3_SDRAM/SDRAM_BA1
- U1 pad Y9: /04_FPGA_Banks2_3_SDRAM/SDRAM_DQM1 -> /04_FPGA_Banks2_3_SDRAM/SDRAM_DQM3
- U7 pad 1: /DF9_CFG-SPW/RST_N -> RST_N
Routing:
- net GND: track 61.3 -> 101.4 mm, vias 35 -> 67
- net VDD3V3: track 75.8 -> 38.2 mm, vias 3 -> 22
- net /05_FPGA_Bank5_SPI/FRAM2_CS_N: track 0.00 -> 26.4 mm, vias 0 -> 1
- net /05_FPGA_Bank5_SPI/FRAM2_MISO: track 0.00 -> 25.6 mm, vias 0 -> 1
- net /04_FPGA_Banks2_3_SDRAM/SDRAM_CS_N: track 48.2 -> 22.7 mm
- net unconnected-(U1D-IO_B5D12P_DQ_SWDO-PadW18): track 0.00 -> 24.2 mm, vias 0 -> 1
- net unconnected-(U1D-IO_B5D12N_DQ_SWDO-PadV18): track 0.00 -> 24.0 mm, vias 0 -> 1
- net unconnected-(U1D-IO_B5D11N_DQ-PadW19): track 0.00 -> 23.0 mm, vias 0 -> 1
- net unconnected-(U1D-IO_B5D11P_DQ-PadY19): track 0.00 -> 22.9 mm, vias 0 -> 1
- net /05_FPGA_Bank5_SPI/FRAM1_CLK: track 0.00 -> 22.1 mm
- net unconnected-(U1D-IO_B5D08N-PadY20): track 0.00 -> 21.5 mm, vias 0 -> 1
- net unconnected-(U1D-IO_B5D14N_DQ_SWDI-PadW17): track 0.00 -> 21.1 mm, vias 0 -> 1
- net unconnected-(U1D-IO_B5D13N_DQS_SWSO-PadY18): track 0.00 -> 20.2 mm, vias 0 -> 1
- net unconnected-(U1D-IO_B5D08P_CLK0-PadY21): track 0.00 -> 20.1 mm, vias 0 -> 1
- net unconnected-(U1D-IO_B5D10N_DQ-PadAA19): track 0.00 -> 19.6 mm, vias 0 -> 1
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
Commit message: added MAX, picoblade, NPN
added the LDO (placement), added the picoblade connector for CFG and deleted one SPW out of 2 in the DF9.
added the NPN transistor (placed)
Parts:
- added J1: Picoblade_CFG, DataHub_Footprints:CONN_532610001-SD_11_MOL, F.Cu at (146.0, 77.1)
- added R20: 1k, Resistor_SMD:R_0402_1005Metric_Pad0.72x0.64mm_HandSolder, F.Cu at (142.9, 72.6)
- added R27: 1k, Resistor_SMD:R_0402_1005Metric_Pad0.72x0.64mm_HandSolder, F.Cu at (120.7, 71.6)
- added R33: 10k, Resistor_SMD:R_0402_1005Metric_Pad0.72x0.64mm_HandSolder, F.Cu at (120.7, 73.6)
- added REF**: LCC-3_STM, DataHub_Footprints:NPN_LCC-3_STM, F.Cu at (172.8, 85.1)
- R31: value 10k -> 1k
- U7, Y2: moved to B.Cu
- moved U7 58.9 mm to (149.8, 77.1), turned to 180 degrees
- turned Y2 to -90 degrees
Connections:
- J3 pad 1: VDD3V3 -> unconnected-(J3-Pad1)
- J3 pad 10: /02_FPGA_Config_JTAG_Bitstream_Reset/SPW2_SOUT_N -> unconnected-(J3-Pad10)
- J3 pad 11: GND -> unconnected-(J3-Pad11)
- J3 pad 12: GND -> unconnected-(J3-Pad12)
- J3 pad 13: /02_FPGA_Config_JTAG_Bitstream_Reset/JTDI -> unconnected-(J3-Pad13)
- J3 pad 14: /02_FPGA_Config_JTAG_Bitstream_Reset/SPW2_SIN_P -> unconnected-(J3-Pad14)
- J3 pad 15: GND -> unconnected-(J3-Pad15)
- J3 pad 16: /02_FPGA_Config_JTAG_Bitstream_Reset/SPW2_SIN_N -> unconnected-(J3-Pad16)
- J3 pad 17: /02_FPGA_Config_JTAG_Bitstream_Reset/JTCK -> unconnected-(J3-Pad17)
- J3 pad 18: GND -> unconnected-(J3-Pad18)
- J3 pad 19: GND -> unconnected-(J3-Pad19)
- J3 pad 2: /02_FPGA_Config_JTAG_Bitstream_Reset/SPW2_DIN_P -> unconnected-(J3-Pad2)
- J3 pad 20: /02_FPGA_Config_JTAG_Bitstream_Reset/SPW2_DOUT_P -> unconnected-(J3-Pad20)
- J3 pad 21: /02_FPGA_Config_JTAG_Bitstream_Reset/JTMS -> unconnected-(J3-Pad21)
- J3 pad 22: /02_FPGA_Config_JTAG_Bitstream_Reset/SPW2_DOUT_N -> unconnected-(J3-Pad22)
- J3 pad 23: GND -> unconnected-(J3-Pad23)
- J3 pad 24: GND -> unconnected-(J3-Pad24)
- J3 pad 25: /02_FPGA_Config_JTAG_Bitstream_Reset/JTRST_N -> unconnected-(J3-Pad25)
- J3 pad 26: /DF9_CFG-SPW/PCLK -> unconnected-(J3-Pad26)
- J3 pad 27: GND -> unconnected-(J3-Pad27)
- J3 pad 28: GND -> unconnected-(J3-Pad28)
- J3 pad 3: GND -> unconnected-(J3-Pad3)
- J3 pad 4: /02_FPGA_Config_JTAG_Bitstream_Reset/SPW2_DIN_N -> unconnected-(J3-Pad4)
- J3 pad 5: RST_N -> unconnected-(J3-Pad5)
- J3 pad 6: GND -> unconnected-(J3-Pad6)
- J3 pad 7: GND -> unconnected-(J3-Pad7)
- J3 pad 8: /02_FPGA_Config_JTAG_Bitstream_Reset/SPW2_SOUT_P -> unconnected-(J3-Pad8)
- J3 pad 9: /02_FPGA_Config_JTAG_Bitstream_Reset/JTDO -> unconnected-(J3-Pad9)
- U1 pad C6: /02_FPGA_Config_JTAG_Bitstream_Reset/SPW2_DOUT_P -> unconnected-(U1F-IO_B12D12P_DQ_SWDO-PadC6)
- U1 pad C7: /02_FPGA_Config_JTAG_Bitstream_Reset/SPW2_DOUT_N -> unconnected-(U1F-IO_B12D12N_DQ_SWDO-PadC7)
- U1 pad F8: /02_FPGA_Config_JTAG_Bitstream_Reset/SPW2_SIN_P -> unconnected-(U1F-IO_B12D15P_DQ_SWSI-PadF8)
- U1 pad G7: /02_FPGA_Config_JTAG_Bitstream_Reset/SPW2_SOUT_P -> unconnected-(U1F-IO_B12D13P_DQS_SWSO-PadG7)
- U1 pad G8: /02_FPGA_Config_JTAG_Bitstream_Reset/SPW2_DIN_P -> unconnected-(U1F-IO_B12D14P_DQ_SWDI-PadG8)
- U1 pad G9: /02_FPGA_Config_JTAG_Bitstream_Reset/SPW2_SIN_N -> unconnected-(U1F-IO_B12D15N_DQ_SWSI-PadG9)
- U1 pad H8: /02_FPGA_Config_JTAG_Bitstream_Reset/SPW2_SOUT_N -> unconnected-(U1F-IO_B12D13N_DQS_SWSO-PadH8)
- U1 pad H9: /02_FPGA_Config_JTAG_Bitstream_Reset/SPW2_DIN_N -> unconnected-(U1F-IO_B12D14N_DQ_SWDI-PadH9)
- U1 pad L8: GND -> /02_FPGA_Config_JTAG_Bitstream_Reset/MODE0
- U1 pad M3: /02_FPGA_Config_JTAG_Bitstream_Reset/PCLK -> Net-(U1G-CLK)
