File: PCB_Project.kicad_pcb (KiCad board)
At the start: 8 copper layers, 152.4 x 101.6 mm, 188 parts, among them J1 Picoblade_CFG, J2 DF9-41P-1V32, J3 DF9-CFG-SPW1, Q1 SOC2222AHRG, Q2 SOC2222AHRG, U1 NX1H35 PBGA625, U10 MAX8556ETE, U11 AS4C8M16SA-6BIN, U2 CY15B108QN-40SXI, U3 CY15B108QN-40SXI, U4 CY15B108QN-40SXI, U5 AS4C8M32S-6TIN, U6 M95P32-IXMNT/E, U7 TPS3828-33DBVR, U8 MAX8556ETE, U9 MAX8556ETE, Y2 LFSPXO025225_25MHz

Commit message: power tree
power tree defined. Few changes remaining but almost finalized
Parts:
- removed Q1, Q2: SOC2222AHRG, DataHub_Footprints:NPN_LCC-3_STM
- removed U10, U8, U9: MAX8556ETE, DataHub_Footprints:MAX8556
- added C111: 10uF, Capacitor_SMD:C_0603_1608Metric_Pad1.08x0.95mm_HandSolder, F.Cu at (234.8, 42.6)
- added C112: 10uF, Capacitor_SMD:C_0603_1608Metric_Pad1.08x0.95mm_HandSolder, F.Cu at (234.8, 45.1)
- added C113: 10uF, Capacitor_SMD:C_0603_1608Metric_Pad1.08x0.95mm_HandSolder, F.Cu at (234.8, 47.6)
- added C114: 10uF, Capacitor_SMD:C_0603_1608Metric_Pad1.08x0.95mm_HandSolder, F.Cu at (234.8, 50.1)
- added C115: 10uF, Capacitor_SMD:C_0603_1608Metric_Pad1.08x0.95mm_HandSolder, F.Cu at (234.8, 52.6)
- added C116: 10uF, Capacitor_SMD:C_0603_1608Metric_Pad1.08x0.95mm_HandSolder, F.Cu at (239.1, 42.6)
- added C117: 10uF, Capacitor_SMD:C_0603_1608Metric_Pad1.08x0.95mm_HandSolder, F.Cu at (239.1, 45.1)
- added C118: 10uF, Capacitor_SMD:C_0603_1608Metric_Pad1.08x0.95mm_HandSolder, F.Cu at (239.1, 47.6)
- added C119: 10uF, Capacitor_SMD:C_0603_1608Metric_Pad1.08x0.95mm_HandSolder, F.Cu at (239.1, 50.1)
- added C120: 10uF, Capacitor_SMD:C_0603_1608Metric_Pad1.08x0.95mm_HandSolder, F.Cu at (239.1, 52.6)
- added C121: 10uF, Capacitor_SMD:C_0603_1608Metric_Pad1.08x0.95mm_HandSolder, F.Cu at (243.5, 42.6)
- added C122: 10uF, Capacitor_SMD:C_0603_1608Metric_Pad1.08x0.95mm_HandSolder, F.Cu at (243.5, 45.1)
- added C123: 10uF, Capacitor_SMD:C_0603_1608Metric_Pad1.08x0.95mm_HandSolder, F.Cu at (243.5, 47.6)
- added C124: 10uF, Capacitor_SMD:C_0603_1608Metric_Pad1.08x0.95mm_HandSolder, F.Cu at (243.5, 50.1)
- added C125: 10uF, Capacitor_SMD:C_0603_1608Metric_Pad1.08x0.95mm_HandSolder, F.Cu at (243.5, 52.6)
- added C126: 10uF, Capacitor_SMD:C_0603_1608Metric_Pad1.08x0.95mm_HandSolder, F.Cu at (247.8, 42.6)
- added C127: 4.7nF, Capacitor_SMD:C_0603_1608Metric_Pad1.08x0.95mm_HandSolder, F.Cu at (247.8, 45.1)
- added C128: 10uF, Capacitor_SMD:C_0603_1608Metric_Pad1.08x0.95mm_HandSolder, F.Cu at (247.8, 47.6)
- added C129: 4.7nF, Capacitor_SMD:C_0603_1608Metric_Pad1.08x0.95mm_HandSolder, F.Cu at (247.8, 50.1)
- added C130: 10uF, Capacitor_SMD:C_0603_1608Metric_Pad1.08x0.95mm_HandSolder, F.Cu at (247.8, 52.6)
- added R44: 100k, Resistor_SMD:R_0402_1005Metric_Pad0.72x0.64mm_HandSolder, F.Cu at (240.9, 54.9)
- added R45: 100k, Resistor_SMD:R_0402_1005Metric_Pad0.72x0.64mm_HandSolder, F.Cu at (240.9, 56.9)
- added R47: 3k74, Resistor_SMD:R_0402_1005Metric_Pad0.72x0.64mm_HandSolder, F.Cu at (240.9, 58.9)
- added R48: 4k02, Resistor_SMD:R_0402_1005Metric_Pad0.72x0.64mm_HandSolder, F.Cu at (240.9, 60.8)
- added R49: 1k, Resistor_SMD:R_0402_1005Metric_Pad0.72x0.64mm_HandSolder, F.Cu at (240.9, 62.8)
- added R50: 1k4, Resistor_SMD:R_0402_1005Metric_Pad0.72x0.64mm_HandSolder, F.Cu at (244.1, 54.9)
- added R51: 1k, Resistor_SMD:R_0402_1005Metric_Pad0.72x0.64mm_HandSolder, F.Cu at (244.1, 56.9)
- added R52: 4k02, Resistor_SMD:R_0402_1005Metric_Pad0.72x0.64mm_HandSolder, F.Cu at (244.1, 58.9)
- added R53: 1k, Resistor_SMD:R_0402_1005Metric_Pad0.72x0.64mm_HandSolder, F.Cu at (244.1, 60.8)
- added R54: 1k2, Resistor_SMD:R_0402_1005Metric_Pad0.72x0.64mm_HandSolder, F.Cu at (244.1, 62.8)
- added R55: 3k74, Resistor_SMD:R_0402_1005Metric_Pad0.72x0.64mm_HandSolder, F.Cu at (247.4, 54.9)
- added R56: 1k2, Resistor_SMD:R_0402_1005Metric_Pad0.72x0.64mm_HandSolder, F.Cu at (247.4, 56.9)
- added R57: 100k, Resistor_SMD:R_0402_1005Metric_Pad0.72x0.64mm_HandSolder, F.Cu at (247.4, 58.9)
- added REF**: RGW0020A, DataHub_Footprints:TPS74201, F.Cu at (190.8, 80.4)
- added U12: MAX8556ETE, DataHub_Footprints:MAX8556, F.Cu at (172.8, 97.9)
- added U13: MAX8556ETE, DataHub_Footprints:MAX8556, F.Cu at (172.7, 87.7)
- added U14: MAX8556ETE, DataHub_Footprints:MAX8556, F.Cu at (163.8, 68.8)
- added U15: TPS74201RGWR, DataHub_Footprints:TPS74201, F.Cu at (172.4, 70.0)
- added U16: TPS74201RGWR, DataHub_Footprints:TPS74201, F.Cu at (171.1, 77.6)
- C51, R10: moved to B.Cu
- moved C45 107.2 mm to (100.4, 24.8)
- moved C52 107.2 mm to (100.4, 27.3)
- moved C53 107.2 mm to (100.4, 29.8)
- moved C54 107.2 mm to (100.4, 32.3)
- moved C55 107.2 mm to (104.7, 24.8)
- moved C56 107.2 mm to (104.7, 27.3)
- moved C57 107.2 mm to (104.7, 29.8)
- moved C58 107.2 mm to (104.7, 32.3)
- moved C59 107.2 mm to (106.3, 44.3)
- moved C61 107.2 mm to (109.1, 24.8)
- moved C63 107.2 mm to (109.1, 27.3)
- moved C81 107.2 mm to (109.1, 29.8)
- moved C97 107.2 mm to (109.1, 32.3)
- moved R34 107.2 mm to (99.8, 34.6)
- moved R35 107.2 mm to (99.8, 36.6)
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Connections:
- net /01_FPGA_Power_Core_PLL/VPL0 renamed /FPGA_Core_PLL/VPL0
- net /01_FPGA_Power_Core_PLL/VPL1 renamed /FPGA_Core_PLL/VPL1
- net /01_FPGA_Power_Core_PLL/VPL2 renamed /FPGA_Core_PLL/VPL2
- net /01_FPGA_Power_Core_PLL/VPL3 renamed /FPGA_Core_PLL/VPL3
- net /02_FPGA_Banks11_12_CFG/CFG_EEPROM_CLK renamed /FPGA_Banks11_12_CFG/CFG_EEPROM_CLK
- net /02_FPGA_Banks11_12_CFG/CFG_EEPROM_CS_N renamed /FPGA_Banks11_12_CFG/CFG_EEPROM_CS_N
- net /02_FPGA_Banks11_12_CFG/CFG_EEPROM_MISO renamed /FPGA_Banks11_12_CFG/CFG_EEPROM_MISO
- net /02_FPGA_Banks11_12_CFG/CFG_EEPROM_MOSI renamed /FPGA_Banks11_12_CFG/CFG_EEPROM_MOSI
- net /02_FPGA_Banks11_12_CFG/JTCK renamed /Connectors_DF9_PICO/JTCK
- net /02_FPGA_Banks11_12_CFG/JTDI renamed /Connectors_DF9_PICO/JTDI
- net /02_FPGA_Banks11_12_CFG/JTDO renamed /Connectors_DF9_PICO/JTDO
- net /02_FPGA_Banks11_12_CFG/JTMS renamed /Connectors_DF9_PICO/JTMS
- net /02_FPGA_Banks11_12_CFG/JTRST_N renamed /Connectors_DF9_PICO/JTRST_N
- net /02_FPGA_Banks11_12_CFG/LD_CFG0 renamed /FPGA_Banks11_12_CFG/LD_CFG0
- net /02_FPGA_Banks11_12_CFG/LD_CFG1 renamed /FPGA_Banks11_12_CFG/LD_CFG1
- net /02_FPGA_Banks11_12_CFG/LD_CFG2 renamed /FPGA_Banks11_12_CFG/LD_CFG2
- net /02_FPGA_Banks11_12_CFG/LD_CFG3 renamed /FPGA_Banks11_12_CFG/LD_CFG3
- net /02_FPGA_Banks11_12_CFG/MODE0 renamed /Connectors_DF9_PICO/MODE0
- net /02_FPGA_Banks11_12_CFG/MODE1 renamed /Connectors_DF9_PICO/MODE1
- net /02_FPGA_Banks11_12_CFG/OSC0 renamed /FPGA_Banks11_12_CFG/OSC0
- net /02_FPGA_Banks11_12_CFG/PERR renamed /FPGA_Banks11_12_CFG/PERR
- net /02_FPGA_Banks11_12_CFG/PRDY renamed /FPGA_Banks11_12_CFG/PRDY
- net /02_FPGA_Banks11_12_CFG/SDRAM_B_A11 renamed /FPGA_Bank10_SDRAMB/SDRAM_B_A11
- net /02_FPGA_Banks11_12_CFG/SDRAM_B_A4 renamed /FPGA_Bank10_SDRAMB/SDRAM_B_A4
- net /02_FPGA_Banks11_12_CFG/SDRAM_B_A5 renamed /FPGA_Bank10_SDRAMB/SDRAM_B_A5
- net /02_FPGA_Banks11_12_CFG/SDRAM_B_A6 renamed /FPGA_Bank10_SDRAMB/SDRAM_B_A6
- net /02_FPGA_Banks11_12_CFG/SDRAM_B_A7 renamed /FPGA_Bank10_SDRAMB/SDRAM_B_A7
- net /02_FPGA_Banks11_12_CFG/SDRAM_B_A8 renamed /FPGA_Bank10_SDRAMB/SDRAM_B_A8
- net /02_FPGA_Banks11_12_CFG/SDRAM_B_A9 renamed /FPGA_Bank10_SDRAMB/SDRAM_B_A9
- net /02_FPGA_Banks11_12_CFG/SDRAM_B_CKE renamed /FPGA_Bank10_SDRAMB/SDRAM_B_CKE
- net /02_FPGA_Banks11_12_CFG/SDRAM_B_CLK renamed /FPGA_Bank10_SDRAMB/SDRAM_B_CLK
- net /02_FPGA_Banks11_12_CFG/SDRAM_B_DQ10 renamed /FPGA_Bank10_SDRAMB/SDRAM_B_DQ10
- net /02_FPGA_Banks11_12_CFG/SDRAM_B_DQ11 renamed /FPGA_Bank10_SDRAMB/SDRAM_B_DQ11
- net /02_FPGA_Banks11_12_CFG/SDRAM_B_DQ12 renamed /FPGA_Bank10_SDRAMB/SDRAM_B_DQ12
- net /02_FPGA_Banks11_12_CFG/SDRAM_B_DQ13 renamed /FPGA_Bank10_SDRAMB/SDRAM_B_DQ13
- net /02_FPGA_Banks11_12_CFG/SDRAM_B_DQ14 renamed /FPGA_Bank10_SDRAMB/SDRAM_B_DQ14
- net /02_FPGA_Banks11_12_CFG/SDRAM_B_DQ15 renamed /FPGA_Bank10_SDRAMB/SDRAM_B_DQ15
- net /02_FPGA_Banks11_12_CFG/SDRAM_B_DQ8 renamed /FPGA_Bank10_SDRAMB/SDRAM_B_DQ8
- net /02_FPGA_Banks11_12_CFG/SDRAM_B_DQ9 renamed /FPGA_Bank10_SDRAMB/SDRAM_B_DQ9
- net /02_FPGA_Banks11_12_CFG/SDRAM_B_UDQM renamed /FPGA_Bank10_SDRAMB/SDRAM_B_UDQM
- net /02_FPGA_Banks11_12_CFG/SPW1_DIN_N renamed /Connectors_DF9_PICO/SPW1_DIN_N
- net /02_FPGA_Banks11_12_CFG/SPW1_DIN_P renamed /Connectors_DF9_PICO/SPW1_DIN_P
- net /02_FPGA_Banks11_12_CFG/SPW1_DOUT_N renamed /Connectors_DF9_PICO/SPW1_DOUT_N
- net /02_FPGA_Banks11_12_CFG/SPW1_DOUT_P renamed /Connectors_DF9_PICO/SPW1_DOUT_P
- net /02_FPGA_Banks11_12_CFG/SPW1_SIN_N renamed /Connectors_DF9_PICO/SPW1_SIN_N
- net /02_FPGA_Banks11_12_CFG/SPW1_SIN_P renamed /Connectors_DF9_PICO/SPW1_SIN_P
- net /02_FPGA_Banks11_12_CFG/SPW1_SOUT_N renamed /Connectors_DF9_PICO/SPW1_SOUT_N
- net /02_FPGA_Banks11_12_CFG/SPW1_SOUT_P renamed /Connectors_DF9_PICO/SPW1_SOUT_P
- net /04_FPGA_Banks2_3_SDRAM/SDRAM_A0 renamed /FPGA_Banks2_3_SDRAM/SDRAM_A0
- net /04_FPGA_Banks2_3_SDRAM/SDRAM_A1 renamed /FPGA_Banks2_3_SDRAM/SDRAM_A1
- net /04_FPGA_Banks2_3_SDRAM/SDRAM_A10 renamed /FPGA_Banks2_3_SDRAM/SDRAM_A10
- net /04_FPGA_Banks2_3_SDRAM/SDRAM_A11 renamed /FPGA_Banks2_3_SDRAM/SDRAM_A11
- net /04_FPGA_Banks2_3_SDRAM/SDRAM_A2 renamed /FPGA_Banks2_3_SDRAM/SDRAM_A2
- net /04_FPGA_Banks2_3_SDRAM/SDRAM_A3 renamed /FPGA_Banks2_3_SDRAM/SDRAM_A3
- net /04_FPGA_Banks2_3_SDRAM/SDRAM_A4 renamed /FPGA_Banks2_3_SDRAM/SDRAM_A4
- net /04_FPGA_Banks2_3_SDRAM/SDRAM_A5 renamed /FPGA_Banks2_3_SDRAM/SDRAM_A5
- net /04_FPGA_Banks2_3_SDRAM/SDRAM_A6 renamed /FPGA_Banks2_3_SDRAM/SDRAM_A6
- net /04_FPGA_Banks2_3_SDRAM/SDRAM_A7 renamed /FPGA_Banks2_3_SDRAM/SDRAM_A7
- net /04_FPGA_Banks2_3_SDRAM/SDRAM_A8 renamed /FPGA_Banks2_3_SDRAM/SDRAM_A8
- net /04_FPGA_Banks2_3_SDRAM/SDRAM_A9 renamed /FPGA_Banks2_3_SDRAM/SDRAM_A9
- net /04_FPGA_Banks2_3_SDRAM/SDRAM_BA0 renamed /FPGA_Banks2_3_SDRAM/SDRAM_BA0
- net /04_FPGA_Banks2_3_SDRAM/SDRAM_BA1 renamed /FPGA_Banks2_3_SDRAM/SDRAM_BA1
- net /04_FPGA_Banks2_3_SDRAM/SDRAM_CAS_N renamed /FPGA_Banks2_3_SDRAM/SDRAM_CAS_N
- net /04_FPGA_Banks2_3_SDRAM/SDRAM_CKE renamed /FPGA_Banks2_3_SDRAM/SDRAM_CKE
- net /04_FPGA_Banks2_3_SDRAM/SDRAM_CLK renamed /FPGA_Banks2_3_SDRAM/SDRAM_CLK
- net /04_FPGA_Banks2_3_SDRAM/SDRAM_CS_N renamed /FPGA_Banks2_3_SDRAM/SDRAM_CS_N
- net /04_FPGA_Banks2_3_SDRAM/SDRAM_DQ0 renamed /FPGA_Banks2_3_SDRAM/SDRAM_DQ0
- net /04_FPGA_Banks2_3_SDRAM/SDRAM_DQ1 renamed /FPGA_Banks2_3_SDRAM/SDRAM_DQ1
- net /04_FPGA_Banks2_3_SDRAM/SDRAM_DQ10 renamed /FPGA_Banks2_3_SDRAM/SDRAM_DQ10
- net /04_FPGA_Banks2_3_SDRAM/SDRAM_DQ11 renamed /FPGA_Banks2_3_SDRAM/SDRAM_DQ11
- net /04_FPGA_Banks2_3_SDRAM/SDRAM_DQ12 renamed /FPGA_Banks2_3_SDRAM/SDRAM_DQ12
- net /04_FPGA_Banks2_3_SDRAM/SDRAM_DQ13 renamed /FPGA_Banks2_3_SDRAM/SDRAM_DQ13
- net /04_FPGA_Banks2_3_SDRAM/SDRAM_DQ14 renamed /FPGA_Banks2_3_SDRAM/SDRAM_DQ14
- net /04_FPGA_Banks2_3_SDRAM/SDRAM_DQ15 renamed /FPGA_Banks2_3_SDRAM/SDRAM_DQ15
- net /04_FPGA_Banks2_3_SDRAM/SDRAM_DQ16 renamed /FPGA_Banks2_3_SDRAM/SDRAM_DQ16
- net /04_FPGA_Banks2_3_SDRAM/SDRAM_DQ17 renamed /FPGA_Banks2_3_SDRAM/SDRAM_DQ17
- net /04_FPGA_Banks2_3_SDRAM/SDRAM_DQ18 renamed /FPGA_Banks2_3_SDRAM/SDRAM_DQ18
- net /04_FPGA_Banks2_3_SDRAM/SDRAM_DQ19 renamed /FPGA_Banks2_3_SDRAM/SDRAM_DQ19
- net /04_FPGA_Banks2_3_SDRAM/SDRAM_DQ2 renamed /FPGA_Banks2_3_SDRAM/SDRAM_DQ2
- net /04_FPGA_Banks2_3_SDRAM/SDRAM_DQ20 renamed /FPGA_Banks2_3_SDRAM/SDRAM_DQ20
- net /04_FPGA_Banks2_3_SDRAM/SDRAM_DQ21 renamed /FPGA_Banks2_3_SDRAM/SDRAM_DQ21
- net /04_FPGA_Banks2_3_SDRAM/SDRAM_DQ22 renamed /FPGA_Banks2_3_SDRAM/SDRAM_DQ22
- net /04_FPGA_Banks2_3_SDRAM/SDRAM_DQ23 renamed /FPGA_Banks2_3_SDRAM/SDRAM_DQ23
- net /04_FPGA_Banks2_3_SDRAM/SDRAM_DQ24 renamed /FPGA_Banks2_3_SDRAM/SDRAM_DQ24
- net /04_FPGA_Banks2_3_SDRAM/SDRAM_DQ25 renamed /FPGA_Banks2_3_SDRAM/SDRAM_DQ25
- net /04_FPGA_Banks2_3_SDRAM/SDRAM_DQ26 renamed /FPGA_Banks2_3_SDRAM/SDRAM_DQ26
- net /04_FPGA_Banks2_3_SDRAM/SDRAM_DQ27 renamed /FPGA_Banks2_3_SDRAM/SDRAM_DQ27
- net /04_FPGA_Banks2_3_SDRAM/SDRAM_DQ28 renamed /FPGA_Banks2_3_SDRAM/SDRAM_DQ28
- net /04_FPGA_Banks2_3_SDRAM/SDRAM_DQ29 renamed /FPGA_Banks2_3_SDRAM/SDRAM_DQ29
- net /04_FPGA_Banks2_3_SDRAM/SDRAM_DQ3 renamed /FPGA_Banks2_3_SDRAM/SDRAM_DQ3
- net /04_FPGA_Banks2_3_SDRAM/SDRAM_DQ30 renamed /FPGA_Banks2_3_SDRAM/SDRAM_DQ30
- net /04_FPGA_Banks2_3_SDRAM/SDRAM_DQ31 renamed /FPGA_Banks2_3_SDRAM/SDRAM_DQ31
- net /04_FPGA_Banks2_3_SDRAM/SDRAM_DQ4 renamed /FPGA_Banks2_3_SDRAM/SDRAM_DQ4
- net /04_FPGA_Banks2_3_SDRAM/SDRAM_DQ5 renamed /FPGA_Banks2_3_SDRAM/SDRAM_DQ5
- net /04_FPGA_Banks2_3_SDRAM/SDRAM_DQ6 renamed /FPGA_Banks2_3_SDRAM/SDRAM_DQ6
- net /04_FPGA_Banks2_3_SDRAM/SDRAM_DQ7 renamed /FPGA_Banks2_3_SDRAM/SDRAM_DQ7
- net /04_FPGA_Banks2_3_SDRAM/SDRAM_DQ8 renamed /FPGA_Banks2_3_SDRAM/SDRAM_DQ8
- net /04_FPGA_Banks2_3_SDRAM/SDRAM_DQ9 renamed /FPGA_Banks2_3_SDRAM/SDRAM_DQ9
- net /04_FPGA_Banks2_3_SDRAM/SDRAM_DQM0 renamed /FPGA_Banks2_3_SDRAM/SDRAM_DQM0
- net /04_FPGA_Banks2_3_SDRAM/SDRAM_DQM1 renamed /FPGA_Banks2_3_SDRAM/SDRAM_DQM1
- net /04_FPGA_Banks2_3_SDRAM/SDRAM_DQM2 renamed /FPGA_Banks2_3_SDRAM/SDRAM_DQM2
- net /04_FPGA_Banks2_3_SDRAM/SDRAM_DQM3 renamed /FPGA_Banks2_3_SDRAM/SDRAM_DQM3
- net /04_FPGA_Banks2_3_SDRAM/SDRAM_RAS_N renamed /FPGA_Banks2_3_SDRAM/SDRAM_RAS_N
- net /04_FPGA_Banks2_3_SDRAM/SDRAM_WE_N renamed /FPGA_Banks2_3_SDRAM/SDRAM_WE_N
- net /05_FPGA_Bank5_SPI/FRAM1_CLK renamed /FPGA_Bank5_SPI/FRAM1_CLK
- net /05_FPGA_Bank5_SPI/FRAM1_CS_N renamed /FPGA_Bank5_SPI/FRAM1_CS_N
- net /05_FPGA_Bank5_SPI/FRAM1_MISO renamed /FPGA_Bank5_SPI/FRAM1_MISO
- net /05_FPGA_Bank5_SPI/FRAM1_MOSI renamed /FPGA_Bank5_SPI/FRAM1_MOSI
- net /05_FPGA_Bank5_SPI/FRAM2_CLK renamed /FPGA_Bank5_SPI/FRAM2_CLK
- net /05_FPGA_Bank5_SPI/FRAM2_CS_N renamed /FPGA_Bank5_SPI/FRAM2_CS_N
- net /05_FPGA_Bank5_SPI/FRAM2_MISO renamed /FPGA_Bank5_SPI/FRAM2_MISO
- net /05_FPGA_Bank5_SPI/FRAM2_MOSI renamed /FPGA_Bank5_SPI/FRAM2_MOSI
- net /05_FPGA_Bank5_SPI/FRAM_RO_CLK renamed /FPGA_Bank5_SPI/FRAM_RO_CLK
- net /05_FPGA_Bank5_SPI/FRAM_RO_CS_N renamed /FPGA_Bank5_SPI/FRAM_RO_CS_N
- net /05_FPGA_Bank5_SPI/FRAM_RO_MISO renamed /FPGA_Bank5_SPI/FRAM_RO_MISO
- net /05_FPGA_Bank5_SPI/FRAM_RO_MOSI renamed /FPGA_Bank5_SPI/FRAM_RO_MOSI
- net /05_FPGA_Bank5_SPI/LD_USER1 renamed /FPGA_Bank5_SPI/LD_USER1
- net /05_FPGA_Bank5_SPI/LD_USER2 renamed /FPGA_Bank5_SPI/LD_USER2
- net /05_FPGA_Bank5_SPI/LD_USER3 renamed /FPGA_Bank5_SPI/LD_USER3
- net /05_FPGA_Bank5_SPI/LD_USER4 renamed /FPGA_Bank5_SPI/LD_USER4
- net /07_FPGA_Bank10_SDRAMB/SDRAM_B_A0 renamed /FPGA_Bank10_SDRAMB/SDRAM_B_A0
- net /07_FPGA_Bank10_SDRAMB/SDRAM_B_A1 renamed /FPGA_Bank10_SDRAMB/SDRAM_B_A1
- net /07_FPGA_Bank10_SDRAMB/SDRAM_B_A10 renamed /FPGA_Bank10_SDRAMB/SDRAM_B_A10
- net /07_FPGA_Bank10_SDRAMB/SDRAM_B_A2 renamed /FPGA_Bank10_SDRAMB/SDRAM_B_A2
- net /07_FPGA_Bank10_SDRAMB/SDRAM_B_A3 renamed /FPGA_Bank10_SDRAMB/SDRAM_B_A3
- net /07_FPGA_Bank10_SDRAMB/SDRAM_B_BA0 renamed /FPGA_Bank10_SDRAMB/SDRAM_B_BA0
- net /07_FPGA_Bank10_SDRAMB/SDRAM_B_BA1 renamed /FPGA_Bank10_SDRAMB/SDRAM_B_BA1
- net /07_FPGA_Bank10_SDRAMB/SDRAM_B_CAS_N renamed /FPGA_Bank10_SDRAMB/SDRAM_B_CAS_N
- net /07_FPGA_Bank10_SDRAMB/SDRAM_B_CS_N renamed /FPGA_Bank10_SDRAMB/SDRAM_B_CS_N
- net /07_FPGA_Bank10_SDRAMB/SDRAM_B_DQ0 renamed /FPGA_Bank10_SDRAMB/SDRAM_B_DQ0
- net /07_FPGA_Bank10_SDRAMB/SDRAM_B_DQ1 renamed /FPGA_Bank10_SDRAMB/SDRAM_B_DQ1
- net /07_FPGA_Bank10_SDRAMB/SDRAM_B_DQ2 renamed /FPGA_Bank10_SDRAMB/SDRAM_B_DQ2
- net /07_FPGA_Bank10_SDRAMB/SDRAM_B_DQ3 renamed /FPGA_Bank10_SDRAMB/SDRAM_B_DQ3
- net /07_FPGA_Bank10_SDRAMB/SDRAM_B_DQ4 renamed /FPGA_Bank10_SDRAMB/SDRAM_B_DQ4
- net /07_FPGA_Bank10_SDRAMB/SDRAM_B_DQ5 renamed /FPGA_Bank10_SDRAMB/SDRAM_B_DQ5
- net /07_FPGA_Bank10_SDRAMB/SDRAM_B_DQ6 renamed /FPGA_Bank10_SDRAMB/SDRAM_B_DQ6
- net /07_FPGA_Bank10_SDRAMB/SDRAM_B_DQ7 renamed /FPGA_Bank10_SDRAMB/SDRAM_B_DQ7
- net /07_FPGA_Bank10_SDRAMB/SDRAM_B_LDQM renamed /FPGA_Bank10_SDRAMB/SDRAM_B_LDQM
- net /07_FPGA_Bank10_SDRAMB/SDRAM_B_RAS_N renamed /FPGA_Bank10_SDRAMB/SDRAM_B_RAS_N
- net /07_FPGA_Bank10_SDRAMB/SDRAM_B_WE_N renamed /FPGA_Bank10_SDRAMB/SDRAM_B_WE_N
- C100 pad 1: VDDIO_11 -> VDD3V3
- C101 pad 1: VDDIO_11 -> VDD3V3
- C102 pad 1: VDDIO_10 -> VDD3V3
- C103 pad 1: VDDIO_10 -> VDD3V3
- C104 pad 1: VDDIO_10 -> VDD3V3
- C105 pad 1: VDDIO_10 -> VDD3V3
- C76 pad 1: VDDIO_0 -> VDD3V3
- C77 pad 1: VDDIO_0 -> VDD3V3
- C78 pad 1: VDDIO_0 -> VDD3V3
- C79 pad 1: VDDIO_2 -> VDD3V3
- C80 pad 1: VDDIO_2 -> VDD3V3
- C82 pad 1: VDDIO_2 -> VDD3V3
- C83 pad 1: VDDIO_2 -> VDD3V3
- C84 pad 1: VDDIO_3 -> VDD3V3
- C85 pad 1: VDDIO_3 -> VDD3V3
- C86 pad 1: VDDIO_3 -> VDD3V3
- C87 pad 1: VDDIO_3 -> VDD3V3
- C88 pad 1: VDDIO_5 -> VDD3V3
- C89 pad 1: VDDIO_5 -> VDD3V3
- C90 pad 1: VDDIO_5 -> VDD3V3
- C98 pad 1: VDDIO_11 -> VDD3V3
- C99 pad 1: VDDIO_11 -> VDD3V3
- J2 pad 1: unconnected-(J2-Pad1) -> +1V7_IN
- J2 pad 10: unconnected-(J2-Pad10) -> GND
- J2 pad 11: unconnected-(J2-Pad11) -> +1V7_IN
- J2 pad 12: unconnected-(J2-Pad12) -> GND
- J2 pad 13: unconnected-(J2-Pad13) -> GND
- J2 pad 14: unconnected-(J2-Pad14) -> +5V_IN
- J2 pad 15: unconnected-(J2-Pad15) -> GND
- J2 pad 16: unconnected-(J2-Pad16) -> +5V_IN
- J2 pad 17: unconnected-(J2-Pad17) -> GND
- J2 pad 18: unconnected-(J2-Pad18) -> GND
- J2 pad 19: unconnected-(J2-Pad19) -> +3V3_IN
- J2 pad 2: unconnected-(J2-Pad2) -> +3V6_IN
- J2 pad 20: unconnected-(J2-Pad20) -> GND
- J2 pad 21: unconnected-(J2-Pad21) -> +3V3_IN
- J2 pad 22: unconnected-(J2-Pad22) -> GND
- J2 pad 23: unconnected-(J2-Pad23) -> +3V3_IN
- J2 pad 24: unconnected-(J2-Pad24) -> GND
- J2 pad 25: unconnected-(J2-Pad25) -> +3V3_IN
- J2 pad 26: unconnected-(J2-Pad26) -> /Connectors_DF9_PICO/B5_12N_DF9
- J2 pad 27: unconnected-(J2-Pad27) -> +3V3_IN
- J2 pad 28: unconnected-(J2-Pad28) -> /Connectors_DF9_PICO/B5_12P_DF9
- J2 pad 29: unconnected-(J2-Pad29) -> GND
- J2 pad 3: unconnected-(J2-Pad3) -> +1V7_IN
- J2 pad 30: unconnected-(J2-Pad30) -> /Connectors_DF9_PICO/B5_11N_DF9
- J2 pad 31: unconnected-(J2-Pad31) -> /Connectors_DF9_PICO/B5_13N_DF9
- J2 pad 32: unconnected-(J2-Pad32) -> /Connectors_DF9_PICO/B5_11P_DF9
- J2 pad 33: unconnected-(J2-Pad33) -> /Connectors_DF9_PICO/B5_10N_DF9
- J2 pad 34: unconnected-(J2-Pad34) -> /Connectors_DF9_PICO/B5_08N_DF9
- J2 pad 35: unconnected-(J2-Pad35) -> /Connectors_DF9_PICO/B5_10P_DF9
- J2 pad 36: unconnected-(J2-Pad36) -> /Connectors_DF9_PICO/B5_08P_DF9
- J2 pad 37: unconnected-(J2-Pad37) -> /Connectors_DF9_PICO/B5_07N_DF9
- J2 pad 38: unconnected-(J2-Pad38) -> /Connectors_DF9_PICO/B5_03N_DF9
- J2 pad 39: unconnected-(J2-Pad39) -> /Connectors_DF9_PICO/B5_04N_DF9
- J2 pad 4: unconnected-(J2-Pad4) -> +3V6_IN
- J2 pad 40: unconnected-(J2-Pad40) -> /Connectors_DF9_PICO/B5_03P_DF9
- J2 pad 41: unconnected-(J2-Pad41) -> /Connectors_DF9_PICO/B5_09N_DF9
- J2 pad 5: unconnected-(J2-Pad5) -> +1V7_IN
- J2 pad 6: unconnected-(J2-Pad6) -> +3V6_IN
- J2 pad 7: unconnected-(J2-Pad7) -> +1V7_IN
- J2 pad 8: unconnected-(J2-Pad8) -> +3V6_IN
- J2 pad 9: unconnected-(J2-Pad9) -> +1V7_IN
- J3 pad 15: unconnected-(J3-Pad15) -> /Connectors_DF9_PICO/B0_11P_DF9
- J3 pad 17: unconnected-(J3-Pad17) -> /Connectors_DF9_PICO/B0_09N_DF9
- J3 pad 18: unconnected-(J3-Pad18) -> /Connectors_DF9_PICO/B0_06P_DF9
- J3 pad 19: unconnected-(J3-Pad19) -> /Connectors_DF9_PICO/B0_05P_DF9
- J3 pad 20: unconnected-(J3-Pad20) -> /Connectors_DF9_PICO/B0_07P_DF9
- J3 pad 21: unconnected-(J3-Pad21) -> /Connectors_DF9_PICO/B0_01N_DF9
- J3 pad 22: unconnected-(J3-Pad22) -> /Connectors_DF9_PICO/B0_08P_DF9
- J3 pad 24: unconnected-(J3-Pad24) -> /Connectors_DF9_PICO/B0_03P_DF9
- J3 pad 25: unconnected-(J3-Pad25) -> /Connectors_DF9_PICO/B0_09P_DF9
- J3 pad 26: unconnected-(J3-Pad26) -> /Connectors_DF9_PICO/B0_03N_DF9
- J3 pad 27: unconnected-(J3-Pad27) -> /Connectors_DF9_PICO/B0_06N_DF9
- J3 pad 28: unconnected-(J3-Pad28) -> /Connectors_DF9_PICO/B0_10N_DF9
- J3 pad 29: unconnected-(J3-Pad29) -> /Connectors_DF9_PICO/B0_01P_DF9
- J3 pad 30: unconnected-(J3-Pad30) -> /Connectors_DF9_PICO/B0_02P_DF9
- J3 pad 33: unconnected-(J3-Pad33) -> /Connectors_DF9_PICO/B0_07N_DF9
- J3 pad 34: unconnected-(J3-Pad34) -> /Connectors_DF9_PICO/B0_02N_DF9
- J3 pad 36: unconnected-(J3-Pad36) -> /Connectors_DF9_PICO/B0_04N_DF9
- J3 pad 37: unconnected-(J3-Pad37) -> /Connectors_DF9_PICO/B0_10P_DF9
- J3 pad 40: unconnected-(J3-Pad40) -> /Connectors_DF9_PICO/B0_04P_DF9
- U1 pad A15: VDDIO_10 -> VDD3V3
- U1 pad A9: VDDIO_11 -> VDD3V3
- U1 pad AA19: unconnected-(U1D-IO_B5D10N_DQ-PadAA19) -> /Connectors_DF9_PICO/B5_10N_DF9
- U1 pad AA20: unconnected-(U1D-IO_B5D10P-PadAA20) -> /Connectors_DF9_PICO/B5_10P_DF9
- U1 pad AA21: unconnected-(U1D-IO_B5D07N-PadAA21) -> /Connectors_DF9_PICO/B5_07N_DF9
- U1 pad AA22: unconnected-(U1D-IO_B5D04N_DQ_SWSI-PadAA22) -> /Connectors_DF9_PICO/B5_04N_DF9
- U1 pad AA23: unconnected-(U1D-IO_B5D03N_DQS_SWDI-PadAA23) -> /Connectors_DF9_PICO/B5_03N_DF9
- U1 pad AB20: unconnected-(U1D-IO_B5D09N-PadAB20) -> /Connectors_DF9_PICO/B5_09N_DF9
- U1 pad AB23: unconnected-(U1D-IO_B5D03P_DQS_SWDI-PadAB23) -> /Connectors_DF9_PICO/B5_03P_DF9
- U1 pad AC1: VDDIO_2 -> VDD3V3
- U1 pad AC25: VDDIO_5 -> VDD3V3
- U1 pad AD13: VDDIO_3 -> VDD3V3
- U1 pad AD7: VDDIO_3 -> VDD3V3
- U1 pad AE2: VDDIO_2 -> VDD3V3
- U1 pad AE21: VDDIO_5 -> VDD3V3
- U1 pad AE24: VDDIO_5 -> VDD3V3
- U1 pad AE5: VDDIO_2 -> VDD3V3
- U1 pad AE9: VDDIO_3 -> VDD3V3
- U1 pad B13: VDDIO_10 -> VDD3V3
- U1 pad B19: VDDIO_10 -> VDD3V3
- U1 pad B7: VDDIO_11 -> VDD3V3
- U1 pad D12: VDDIO_11 -> VDD3V3
- U1 pad F1: VDDIO_0 -> VDD3V3
- U1 pad F12: VDDIO_11 -> VDD3V3
- U1 pad G1: unconnected-(U1A-IO_B0D05P-PadG1) -> /Connectors_DF9_PICO/B0_05P_DF9
- U1 pad G3: unconnected-(U1A-IO_B0D08P-PadG3) -> /Connectors_DF9_PICO/B0_08P_DF9
- U1 pad G4: unconnected-(U1A-IO_B0D09P-PadG4) -> /Connectors_DF9_PICO/B0_09P_DF9
- U1 pad G5: unconnected-(U1A-IO_B0D09N-PadG5) -> /Connectors_DF9_PICO/B0_09N_DF9
- U1 pad G6: unconnected-(U1A-IO_B0D11P_CLK1-PadG6) -> /Connectors_DF9_PICO/B0_11P_DF9
- U1 pad H1: unconnected-(U1A-IO_B0D01P-PadH1) -> /Connectors_DF9_PICO/B0_01P_DF9
- U1 pad H13: VDDIO_10 -> VDD3V3
- U1 pad H2: unconnected-(U1A-IO_B0D01N-PadH2) -> /Connectors_DF9_PICO/B0_01N_DF9
- U1 pad H3: unconnected-(U1A-IO_B0D06P-PadH3) -> /Connectors_DF9_PICO/B0_06P_DF9
- U1 pad H4: unconnected-(U1A-IO_B0D06N-PadH4) -> /Connectors_DF9_PICO/B0_06N_DF9
- U1 pad H5: unconnected-(U1A-IO_B0D07P-PadH5) -> /Connectors_DF9_PICO/B0_07P_DF9
- U1 pad H6: unconnected-(U1A-IO_B0D07N-PadH6) -> /Connectors_DF9_PICO/B0_07N_DF9
- U1 pad J1: VDDIO_0 -> VDD3V3
- U1 pad J3: unconnected-(U1A-IO_B0D02P-PadJ3) -> /Connectors_DF9_PICO/B0_02P_DF9
- U1 pad J4: unconnected-(U1A-IO_B0D02N-PadJ4) -> /Connectors_DF9_PICO/B0_02N_DF9
- U1 pad J5: unconnected-(U1A-IO_B0D03P-PadJ5) -> /Connectors_DF9_PICO/B0_03P_DF9
- U1 pad J6: unconnected-(U1A-IO_B0D03N-PadJ6) -> /Connectors_DF9_PICO/B0_03N_DF9
- U1 pad J7: unconnected-(U1A-IO_B0D10P_CLK0-PadJ7) -> /Connectors_DF9_PICO/B0_10P_DF9
- U1 pad J8: unconnected-(U1A-IO_B0D10N-PadJ8) -> /Connectors_DF9_PICO/B0_10N_DF9
- U1 pad K7: unconnected-(U1A-IO_B0D04P-PadK7) -> /Connectors_DF9_PICO/B0_04P_DF9
- U1 pad K8: unconnected-(U1A-IO_B0D04N-PadK8) -> /Connectors_DF9_PICO/B0_04N_DF9
- U1 pad L9: VDDIO_0 -> VDD3V3
- U1 pad V17: VDDIO_5 -> VDD3V3
- U1 pad V18: unconnected-(U1D-IO_B5D12N_DQ_SWDO-PadV18) -> /Connectors_DF9_PICO/B5_12N_DF9
- U1 pad V9: VDDIO_2 -> VDD3V3
- U1 pad W13: VDDIO_3 -> VDD3V3
- U1 pad W18: unconnected-(U1D-IO_B5D12P_DQ_SWDO-PadW18) -> /Connectors_DF9_PICO/B5_12P_DF9
- U1 pad W19: unconnected-(U1D-IO_B5D11N_DQ-PadW19) -> /Connectors_DF9_PICO/B5_11N_DF9
- U1 pad Y18: unconnected-(U1D-IO_B5D13N_DQS_SWSO-PadY18) -> /Connectors_DF9_PICO/B5_13N_DF9
- U1 pad Y19: unconnected-(U1D-IO_B5D11P_DQ-PadY19) -> /Connectors_DF9_PICO/B5_11P_DF9
- U1 pad Y20: unconnected-(U1D-IO_B5D08N-PadY20) -> /Connectors_DF9_PICO/B5_08N_DF9
- U1 pad Y21: unconnected-(U1D-IO_B5D08P_CLK0-PadY21) -> /Connectors_DF9_PICO/B5_08P_DF9
Routing:
- net VDD3V3: track 53.8 -> 94.0 mm, vias 33 -> 68
- net /Connectors_DF9_PICO/B0_10P_DF9: track 0.00 -> 30.7 mm, vias 0 -> 2
- net /Connectors_DF9_PICO/B5_12N_DF9: track 0.00 -> 29.3 mm, vias 0 -> 2
- net /Connectors_DF9_PICO/B5_12P_DF9: track 0.00 -> 29.3 mm, vias 0 -> 2
- net /Connectors_DF9_PICO/B5_11P_DF9: track 0.00 -> 27.9 mm, vias 0 -> 2
- net /Connectors_DF9_PICO/B5_11N_DF9: track 0.00 -> 27.9 mm, vias 0 -> 2
- net unconnected-(U1A-IO_B0D10P_CLK0-PadJ7): track 27.3 -> 0.00 mm, vias 1 -> 0
- net /Connectors_DF9_PICO/B0_07N_DF9: track 0.00 -> 27.3 mm, vias 0 -> 2
- net /Connectors_DF9_PICO/B5_08N_DF9: track 0.00 -> 26.4 mm, vias 0 -> 2
- net /Connectors_DF9_PICO/B0_11P_DF9: track 0.00 -> 25.2 mm, vias 0 -> 2
- net /Connectors_DF9_PICO/B5_08P_DF9: track 0.00 -> 25.0 mm, vias 0 -> 2
- net /Connectors_DF9_PICO/B0_09P_DF9: track 0.00 -> 24.3 mm, vias 0 -> 2
- net /Connectors_DF9_PICO/B0_09N_DF9: track 0.00 -> 24.2 mm, vias 0 -> 2
- net /Connectors_DF9_PICO/B0_06N_DF9: track 0.00 -> 24.1 mm, vias 0 -> 2
- net unconnected-(U1A-IO_B0D07N-PadH6): track 24.0 -> 0.00 mm, vias 1 -> 0
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- added copper zone on B.Cu, net +1V7_IN
- added copper zone on F.Cu, net +1V7_IN
- added copper zone on B.Cu, net +3V3_IN
- added copper zone on F.Cu, net +3V3_IN
- added copper zone on In1.Cu, net GND
- added copper zone on In6.Cu, net GND
- added copper zone on F.Cu, net VDD1V2
- added copper zone on In3.Cu, net VDD1V2
- added copper zone on F.Cu, net VDD2V5A
- added copper zone on In3.Cu, net VDD2V5A
Other:
- board size 152.4 x 101.6 mm -> 61.3 x 70 mm
