File: FPGA_Bank0_1.kicad_sch (KiCad schematic)
At the start: 24 parts, among them U1 NX1H35 PBGA625, U2 M95P32-IXMNT/E, Y1 LFSPXO025225_25MHz

Commit message: pre order checks
ADDED jumper for VDDSENSE remote sensing / 1V2 core PWR for MAX LDO feedback
Parts:
- removed C13, C14, C97: 100nF, Capacitor_SMD:C_0402_1005Metric_Pad0.74x0.62mm_HandSolder, symbol Device:C_Small
- removed D1, D2, D3, D4, D6: LED_green, LED_SMD:LED_0603_1608Metric, symbol Device:LED_Small
- removed D5: LED_red, LED_SMD:LED_0603_1608Metric, symbol Device:LED_Small
- removed L5: 10uH, Inductor_SMD:L_0603_1608Metric_Pad1.05x0.95mm_HandSolder, symbol Device:L_Small
- removed R1, R10, R11, R2, R6, R7, R8, R9: 1k, Resistor_SMD:R_0402_1005Metric_Pad0.72x0.64mm_HandSolder, symbol Device:R_Small
- removed R3, R4: 10k, Resistor_SMD:R_0402_1005Metric_Pad0.72x0.64mm_HandSolder, symbol Device:R_Small
- removed R5: 100k, Resistor_SMD:R_0402_1005Metric_Pad0.72x0.64mm_HandSolder, symbol Device:R_Small
- removed U1: NX1H35 PBGA625, DataHub_NG_Medium:NX1H35S_CLGA625, symbol Brave625:root_0_BRAVE625A_Brave625.SchLib
- removed U2: M95P32-IXMNT/E, DataHub_Footprints:SO8N_4X5X1P27_STM, symbol Memory_EEPROM:25LCxxx-MF
- removed Y1: LFSPXO025225_25MHz, DataHub_Footprints:SON4_LFSPXO025225_IQD-M, symbol Oscillator:ASCO
- added U1: NX1H35 PBGA625, DataHub_NG_Medium:NX1H35S_CLGA625, symbol Brave625:root_0_BRAVE625A_Brave625.SchLib
Connections:
- net GND: now also U1.F2 (GNDIO_0), U1.F24 (GNDIO_8), U1.F25 (VDDIO_8), U1.J2 (GNDIO_0), U1.J25 (VDDIO_8), U1.K17 (GNDIO_8), U1.K18 (VDDIO_8), U1.K24 (GNDIO_8), U1.K9 (GNDIO_0), U1.L24 (GNDIO_7), U1.L25 (VDDIO_7), U1.R22 (VDDIO_7), U1.R23 (GNDIO_7), U1.R24 (GNDIO_7), U1.R25 (VDDIO_7), U1.R9 (GNDIO_1), U1.T9 (VDDIO_1), U1.U1 (VDDIO_1), U1.U2 (GNDIO_1), U1.Y1 (VDDIO_1), U1.Y2 (GNDIO_1)
- new net B0_01N_DF9: U1.H2 (IO_B0D01N)
- new net B0_01P_DF9: U1.H1 (IO_B0D01P)
- new net B0_02N_DF9: U1.J4 (IO_B0D02N)
- new net B0_02P_DF9: U1.J3 (IO_B0D02P)
- new net B0_03N_DF9: U1.J6 (IO_B0D03N)
- new net B0_03P_DF9: U1.J5 (IO_B0D03P)
- new net B0_04N_DF9: U1.K8 (IO_B0D04N)
- new net B0_04P_DF9: U1.K7 (IO_B0D04P)
- new net B0_05P_DF9: U1.G1 (IO_B0D05P)
- new net B0_06N_DF9: U1.H4 (IO_B0D06N)
- new net B0_06P_DF9: U1.H3 (IO_B0D06P)
- new net B0_07N_DF9: U1.H6 (IO_B0D07N)
- new net B0_07P_DF9: U1.H5 (IO_B0D07P)
- new net B0_08P_DF9: U1.G3 (IO_B0D08P)
- new net B0_09N_DF9: U1.G5 (IO_B0D09N)
- new net B0_09P_DF9: U1.G4 (IO_B0D09P)
- new net B0_10N_DF9: U1.J8 (IO_B0D10N)
- new net B0_10P_DF9: U1.J7 (IO_B0D10P_CLK0)
- new net B0_11P_DF9: U1.G6 (IO_B0D11P_CLK1)
- new net VDDIO_0: U1.F1 (VDDIO_0), U1.J1 (VDDIO_0), U1.L9 (VDDIO_0)
- no-connect marks 87 -> 85
Other:
- note added: "Bank 0: spare user I/Os routed to the DF9 board-to-board connector."
- note added: "Bank 1: unused"
- note added: "FPGA Banks 0 and 1"
- note added: "FPGA Banks 7 and 8 (unused)"
- note removed: "25MHz oscillator used for system clock."
- note removed: "Bank 11: connected to the secondary BGA SDRAM interface."
- note removed: "Bank 12: connected to the SpaceWire interface and the 25 MHz oscillator clock input."
- note removed: "Bank 6: unused"
- note removed: "Bank SERVICE: dedicated to FPGA configuration, programming, reset, and service interfaces."
- note removed: "CFG EEPROM"
- note removed: "FPGA Banks 11 and 12"
- note removed: "FPGA Banks 6 and SERVICE"
- note removed: "LEDs"
- note removed: "Oscillator"
- note removed: "Stores the FPGA configuration bitstream. Used during power-up for Master SPI configuration."
- note removed: "Visual indicators for the PRDY and PERR programming/status signals."
- company: (none) -> KTH Royal Institute of Technology
- title: (none) -> FPGA Banks 0 and 1
