File: FPGA_Banks11_12_CFG_Service.kicad_sch (KiCad schematic)
At the start: 24 parts, among them U1 NX1H35 PBGA625, U2 M95P32-IXMNT/E, Y1 LFSPXO025225_25MHz

Commit message: pre order checks
ADDED jumper for VDDSENSE remote sensing / 1V2 core PWR for MAX LDO feedback
Other:
- company: (none) -> KTH Royal Institute of Technology
- title: (none) -> FPGA Configuration, Service and Banks 11-12
Changed lines of the file:
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@@
 	(generator_version "9.0")
 	(paper "A3")
+	(title_block
+		(title "FPGA Configuration, Service and Banks 11-12")
+		(date "2026-10-06")
+		(rev "1.0")
+		(company "KTH Royal Institute of Technology")
+	)
 	(rectangle
 		(start 243.84 17.78)
@@
 		)
 		(instances
-			(project ""
+			(project "PCB_Project"
 				(path "/ae14ff2f-b8e3-4dd1-9329-e73906805e39/e4b4090a-9491-4976-8b45-759656425e5b"
 					(reference "#PWR016")
@@
 		)
 		(instances
-			(project ""
+			(project "PCB_Project"
 				(path "/ae14ff2f-b8e3-4dd1-9329-e73906805e39/e4b4090a-9491-4976-8b45-759656425e5b"
 					(reference "#PWR030")
