File: FPGA_Banks2_3_SDRAM.kicad_sch (KiCad schematic)
At the start: 6 parts, among them U1 NX1H35 PBGA625, U3 AS4C8M32S-6TIN

Commit message: pre order checks
ADDED jumper for VDDSENSE remote sensing / 1V2 core PWR for MAX LDO feedback
Other:
- company: (none) -> KTH Royal Institute of Technology
- title: (none) -> Primary SDRAM Interface - FPGA Banks 2 and 3
Changed lines of the file:
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@@
 	(generator_version "9.0")
 	(paper "A3")
+	(title_block
+		(title "Primary SDRAM Interface - FPGA Banks 2 and 3")
+		(date "2026-10-06")
+		(rev "1.0")
+		(company "KTH Royal Institute of Technology")
+	)
 	(rectangle
 		(start 43.18 27.94)
@@
 		)
 		(instances
-			(project ""
+			(project "PCB_Project"
 				(path "/ae14ff2f-b8e3-4dd1-9329-e73906805e39/3e72565b-8456-42ee-89da-a690bc2340a4"
 					(reference "#PWR047")
@@
 		)
 		(instances
-			(project ""
+			(project "PCB_Project"
 				(path "/ae14ff2f-b8e3-4dd1-9329-e73906805e39/3e72565b-8456-42ee-89da-a690bc2340a4"
 					(reference "#PWR045")
