File: FPGA_Banks9_10_SDRAM_bga.kicad_sch (KiCad schematic)
At the start: 6 parts, among them U1 NX1H35 PBGA625, U4 AS4C8M16SA-6BIN

Commit message: pre order checks
ADDED jumper for VDDSENSE remote sensing / 1V2 core PWR for MAX LDO feedback
Other:
- company: (none) -> KTH Royal Institute of Technology
- title: (none) -> Secondary SDRAM Interface - FPGA Banks 9 and 10
Changed lines of the file:
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@@
 	(generator_version "9.0")
 	(paper "A3")
+	(title_block
+		(title "Secondary SDRAM Interface - FPGA Banks 9 and 10")
+		(date "2026-10-06")
+		(rev "1.0")
+		(company "KTH Royal Institute of Technology")
+	)
 	(rectangle
 		(start 209.55 39.116)
@@
 		)
 		(instances
-			(project ""
+			(project "PCB_Project"
 				(path "/ae14ff2f-b8e3-4dd1-9329-e73906805e39/43ca8a3e-d0ec-4d1b-80e5-099bf8df79e9"
 					(reference "U4")
